File: board/6502__R8_EXP1.sch (EAGLE design)
At the start: 19 parts, among them IC2 74HCT02N, IC3 74HCT04N, IC4 74HCT373N, IC5 74HCT02N, IC6 74HCT244N

Commit message: Expansion board: Improve Layout, Fix Errors
Parts:
- added C16: 1u, rcl:CPOL-EUE5-5
- added C18: 100n, rcl:C-EU025-030X050
- added C19: 10u, rcl:CPOL-EUE5-5
- added C20: 220u, rcl:CPOL-EUE5-5
- added C21: 47n, rcl:C-EU025-030X050
- added IC16: LM386N-3, linear:LM386N-3
- added IC7: MEGA32-A, atmel:MEGA32-A
- added JP4: (no value), pinhead:PINHD-1X1
- added JP5: (no value), pinhead:PINHD-1X3
- added JP6, JP7: (no value), pinhead:PINHD-1X8
- added R10: 10R, rcl:R-EU_0207/12
- added R7: 1k, rcl:R-EU_0207/12
- added R8: 10k, rcl:R-EU_0207/12
- added R9: 1k2, rcl:R-EU_0207/12
- added SV3: (no value), con-lstb:MA08-1
- added SV4: (no value), con-lstb:MA20-1
- added SV5: (no value), con-lstb:MA03-2
- added X1: TOBU3, logik2:TOBU3
- U$2: device logik:SOLDERPAD -> logik2:SOLDERPAD
Connections:
- new net N$114: JP5.1, JP5.2, JP5.3, R7.2, R8.1
- new net N$115: C16.+, R8.2
- new net N$116: C16.-, IC16.+IN
- new net N$117: C18.1, IC16.BYPASS
- new net N$126: C19.-, IC16.GAIN@2
- new net N$127: IC16.GAIN@1, R9.2
- new net N$128: C19.+, R9.1
- new net N$129: C20.-, X1.1
- new net N$130: C20.+, C21.1, IC16.OUT
- new net N$133: C21.2, R10.1
- new net N$31: IC1.IOB0, JP6.1
- new net N$32: IC7.(ADC0)PA0, SV3.1
- new net N$33: IC7.(ADC1)PA1, SV3.2
- new net N$34: IC7.(ADC2)PA2, SV3.3
- new net N$35: IC7.(RXD)PD0, SV4.20
- new net N$36: IC7.(TXD)PD1, SV4.19
- new net N$37: IC7.(INT0)PD2, SV4.18
- new net N$38: IC7.(INT1)PD3, SV4.17
- new net N$39: IC7.(OC1B)PD4, SV4.16
- new net N$40: IC7.(OC1A)PD5, SV4.15
- new net N$41: IC7.(ICP)PD6, SV4.14
- new net N$42: IC7.(OC2)PD7, SV4.13
- new net N$43: IC7.PC0(SCL), SV4.12
- new net N$44: IC7.PC1(SDA), SV4.11
- new net N$45: IC7.(TCK)PC2, SV4.10
- new net N$46: IC7.(TMS)PC3, SV4.9
- new net N$47: IC7.(TDO)PC4, SV4.8
- new net N$48: IC7.(TDI)PC5, SV4.7
- new net N$49: IC7.(TOSC1)PC6, SV4.6
- new net N$50: IC7.(TOSC2)PC7, SV4.5
- new net N$51: IC7.(MISO)PB6, SV5.1
- new net N$52: IC7.(SCK)PB7, SV5.3
- new net N$53: IC7.(ADC3)PA3, SV3.4
- new net N$54: IC7.(MOSI)PB5, SV5.4
- new net N$55: IC7.(ADC4)PA4, SV3.5
- new net N$56: IC7.(ADC5)PA5, SV3.6
- new net N$57: IC7.(ADC6)PA6, SV3.7
- new net N$58: IC7.(ADC7)PA7, SV3.8
- new net N$59: IC1.IOB1, JP6.2
- new net N$60: IC1.IOB2, JP6.3
- new net N$61: IC1.IOB3, JP6.4
- new net N$62: IC1.IOB4, JP6.5
- new net N$63: IC1.IOB5, JP6.6
- new net N$64: IC1.IOB6, JP6.7
- new net N$65: IC1.IOB7, JP6.8
- new net N$66: IC1.IOA0, JP7.1
- new net N$67: IC1.IOA1, JP7.2
- new net N$68: IC1.IOA2, JP7.3
- new net N$69: IC1.IOA3, JP7.4
- new net N$70: IC1.IOA4, JP7.5
- new net N$71: IC1.IOA5, JP7.6
- new net N$72: IC1.IOA6, JP7.7
- new net N$73: IC1.IOA7, JP7.8
- net !RESET: now also IC7.RESET, SV5.5
- net !VRAM: now also JP4.1
- net VCC: now also IC16.VS, IC4P.VCC, IC6P.VCC, IC7.AREF, IC7.AVCC, IC7.VCC, IC7.VCC1, IC7.VCC2, SV5.2
- net VSS: now also C18.2, IC16.-IN, IC16.GND, IC4P.GND, IC6P.GND, IC7.GND, IC7.GND1, IC7.GND2, IC7.GND@1, R10.2, R7.1, SV5.6, X1.2
Other:
- moved on the sheet: IC3C, IC5B
